Commit message: fixed solar panel only environment

File: urdf/solar.urdf.xacro (robot description, xacro)
@@ -10,5 +10,5 @@
       <origin xyz="0 0 0" rpy="0 0 0"/>
       <geometry>
-        <mesh filename="package://cpr_agriculture_gazebo/meshes/solar2.dae"/>
+        <mesh filename="package://durable_gazebo_simulation/meshes/solar_farm.dae"/>
       </geometry>
     </visual>
@@ -16,5 +16,5 @@
       <origin xyz="0 0 0" rpy="0 0 0"/>
       <geometry>
-        <mesh filename="package://cpr_agriculture_gazebo/meshes/solar2.dae"/>
+        <mesh filename="package://durable_gazebo_simulation/meshes/solar_farm.dae"/>
       </geometry>
     </collision>
